File: hardware/Villa_Hacker_Badge.kicad_sch (KiCad schematic)
At the start: 16 parts, among them J1 Conn_02x03_Odd_Even, SW1 SW_RST, SW2 On, U1 PY32F002AA15M6TU

Commit message: feat(Hw):Added_details
Parts:
- D4: value Purple -> Orange; LCSC# C7371915 -> C84262
Other:
- company: (none) -> Electronic Cats
- title: (none) -> badge_villa
- moved on the sheet: C1, D1, D2, D3, D4, D5, J1, R1, R2, R3, R4, R5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

Commit message: fix (hw): update #LCSC orange LED
Parts:
- D4: LCSC# C84262 -> C434437
Changed lines of the file:
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@@
 			)
 		)
-		(property "LCSC#" "C84262"
+		(property "LCSC#" "C434437"
 			(at 183.896 91.186 0)
 			(effects
