File: hardware/Villa_Hacker_Badge.kicad_pcb (KiCad board)
At the start: 2 copper layers, 45.1 x 50 mm, 17 parts, among them J1 Conn_02x03_Odd_Even, SW1 SW_RST, SW2 On, U1 PY32F002AA15M6TU

Commit message: feat(Hw):Added_details
Parts:
- added kibuzzard-66857BF8: G***, kibuzzard-66857BF8, B.Cu at (84.4, 74.5)
- added kibuzzard-66857C28: G***, kibuzzard-66857C28, B.Cu at (84.1, 66.8)
- added kibuzzard-66858654: G***, kibuzzard-66858654, B.Cu at (89.7, 74.4)
- added kibuzzard-66858661: G***, kibuzzard-66858661, B.Cu at (89.4, 66.8)
- D4: value Purple -> Orange
- moved J1 5.26 mm to (89.5, 71.9), turned to 90 degrees
- moved R4 3.13 mm to (93.3, 44.2)
- moved R3 2.50 mm to (64.7, 43.3)
- turned C1 to 180 degrees
Routing:
- net GND: track 71.9 -> 54.6 mm
- net +3.3V: track 59.9 -> 73.7 mm
- net /SWDIO: track 15.7 -> 28.1 mm
- net /SWCLK: track 19.7 -> 24.2 mm
- net Net-(D4-K): track 4.69 -> 7.04 mm
- net Net-(D3-K): track 3.41 -> 5.47 mm
- net /PA1: track 43.5 -> 44.2 mm
- net /PF0: track 31.7 -> 31.1 mm
- removed copper zone on F.Cu, net (none)

Commit message: feat(hw): add labels and logos
Parts:
- added G***: LOGO, Aesthetics:electronic_cats_logo_4x3, B.Cu at (68.1, 62.8)
- added kibuzzard-6685884A: G***, kibuzzard-6685884A, B.Cu at (87.8, 61.2)
- added kibuzzard-668588B5: G***, kibuzzard-668588B5, B.Cu at (68.5, 67.6)
Other:
- board text added: "¡Lengua de toda mi raza, habla de plata y cristal, ardiente como una llama, viva cual un manantial! Juana de Ibarbourou"

Commit message: feat(Hw):Add_Hole
Parts:
- moved D1 0.42 mm to (92.5, 50.6)
Routing:
- net GND: track 54.6 -> 75.2 mm, vias 4 -> 11
- net /PA6: track 13.6 -> 9.73 mm
Other:
- outline, holes or cut-outs redrawn
